Commit message: testing multiple urdfs

File: description/target_description.urdf (robot description, URDF)
Before this commit: robot target, 1 links, 0 joints
Links:
- removed link base_link
- added link target_link; visual box size=${code_length} ${code_length} 0.001
- added link target_zone_1_link
Joints:
- added joint target_zone_1_joint: type fixed, parent target_link, child target_zone_1_link, origin xyz=1 0 0

Commit message: added extra link

File: description/target_description.urdf (robot description, URDF)
Before this commit: robot target, 2 links, 1 joints
Links:
- added link table_tag
- link target_link: geometry visual box size=${code_length} ${code_length} 0.1
Joints:
- added joint april_tag_joint: type fixed, parent table_tag, child target_link, origin xyz=0 0 0

Commit message: progress

File: description/target_description.urdf (robot description, URDF)
Before this commit: robot target, 3 links, 2 joints
Joints:
- joint april_tag_joint: origin xyz=0 0 0 -> xyz=0 0 0 rpy=0 0 0
- joint target_zone_1_joint: origin xyz=1 0 0 -> xyz=0.3 0 0 rpy=0 0 ${pi/2}

Commit message: finish hooking v2

File: description/target_description.urdf (robot description, URDF)
Before this commit: robot target, 3 links, 2 joints
Joints:
- joint target_zone_1_joint: origin xyz=0.3 0 0 rpy=0 0 ${pi/2} -> xyz=0.25 -0.2 0 rpy=0 0 ${pi/2}

Commit message: added new targets to description

File: description/target_description.urdf (robot description, URDF)
Before this commit: robot target, 3 links, 2 joints
Links:
- added link target_zone_0_link
- added link target_zone_2_link
Joints:
- added joint target_zone_0_joint: type fixed, parent target_link, child target_zone_0_link, origin xyz=0.25 -0.2 0 rpy=0 0 ${pi/2}
- added joint target_zone_2_joint: type fixed, parent target_link, child target_zone_2_link, origin xyz=-0.25 -0.2 0 rpy=0 0 ${-pi/2}
- joint target_zone_1_joint: origin xyz=0.25 -0.2 0 rpy=0 0 ${pi/2} -> xyz=-0.25 -0.2 0 rpy=0 0 ${pi/2}
